File: faults.sch (KiCad schematic (older format))
At the start: 93 parts

Commit message: rename stuff
Parts:
- UA? (x4): symbol wind_components:TL331 -> turbine_components:TL331
Changed lines of the file:
@@
 $EndComp
 $Comp
-L wind_components:TL331 UA?
+L turbine_components:TL331 UA?
 U 1 1 6480480D
 P 5350 3600
@@
 $EndComp
 $Comp
-L wind_components:TL331 UA?
+L turbine_components:TL331 UA?
 U 1 1 64804855
 P 2100 1750
@@
 Connection ~ 950  3950
 $Comp
-L wind_components:TL331 UA?
+L turbine_components:TL331 UA?
 U 1 1 648048CB
 P 4900 1800
@@
 $EndComp
 $Comp
-L wind_components:TL331 UA?
+L turbine_components:TL331 UA?
 U 1 1 64804995
 P 5350 5000
